File: uPlaits_SE_Assembly_Template.brd (EAGLE design)
At the start: 40 x 110.5 mm, 0 parts

Commit message: Revision B
Parts:
- added E$1, E$2: (no value), uPlaits_SE_Library:HOLE-M2.5
Routing:
- added copper zone on layer 1, net GND
- added copper zone on layer 16, net GND
Other:
- board text added: "2.0 mm"
- board text added: "2021-01-01 tall-dog.com"
- board text added: "TD-UPSE-C-AT"
- board text added: "µPlaits SE Assembly Template"
- board text removed: "µPlaits SE Assembly Template TD-UPSE-B-AT CC BY-SA 4.0 2019-01-17 tall-dog.com"
Changed lines of the file:
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@@
 <?xml version="1.0" encoding="utf-8"?>
 <!DOCTYPE eagle SYSTEM "eagle.dtd">
-<eagle version="9.3.0">
+<eagle version="9.6.2">
 <drawing>
 <settings>
@@
 <layers>
 <layer number="1" name="Top" color="4" fill="1" visible="yes" active="yes"/>
+<layer number="2" name="Route2" color="1" fill="3" visible="no" active="no"/>
+<layer number="15" name="Route15" color="4" fill="6" visible="no" active="no"/>
 <layer number="16" name="Bottom" color="1" fill="1" visible="yes" active="yes"/>
 <layer number="17" name="Pads" color="2" fill="1" visible="yes" active="yes"/>
@@
 <layer number="20" name="Dimension" color="24" fill="1" visible="yes" active="yes"/>
 <layer number="21" name="tPlace" color="7" fill="1" visible="yes" active="yes"/>
-<layer number="22" name="bPlace" color="7" fill="1" visible="yes" active="yes"/>
+<layer number="22" name="bPlace" color="14" fill="1" visible="yes" active="yes"/>
 <layer number="23" name="tOrigins" color="15" fill="1" visible="yes" active="yes"/>
 <layer number="24" name="bOrigins" color="15" fill="1" visible="yes" active="yes"/>
@@
 <layer number="51" name="tDocu" color="7" fill="1" visible="yes" active="yes"/>
 <layer number="52" name="bDocu" color="7" fill="1" visible="yes" active="yes"/>
+<layer number="88" name="SimResults" color="9" fill="1" visible="no" active="no"/>
+<layer number="89" name="SimProbes" color="9" fill="1" visible="no" active="no"/>
+<layer number="90" name="Modules" color="5" fill="1" visible="no" active="no"/>
+<layer number="91" name="Nets" color="2" fill="1" visible="no" active="no"/>
+<layer number="92" name="Busses" color="1" fill="1" visible="no" active="no"/>
+<layer number="93" name="Pins" color="2" fill="1" visible="no" active="no"/>
+<layer number="94" name="Symbols" color="4" fill="1" visible="no" active="no"/>
+<layer number="95" name="Names" color="7" fill="1" visible="no" active="no"/>
+<layer number="96" name="Values" color="7" fill="1" visible="no" active="no"/>
+<layer number="97" name="Info" color="7" fill="1" visible="no" active="no"/>
+<layer number="98" name="Guide" color="6" fill="1" visible="no" active="no"/>
 </layers>
 <board>
@@
 <wire x1="40" y1="3" x2="37" y2="0" width="0" layer="20" curve="-90"/>
 <wire x1="37" y1="110.5" x2="40" y2="107.5" width="0" layer="20" curve="-90"/>
-<text x="20" y="29" size="1.5" layer="21" ratio="10" align="center">µPlaits SE
-Assembly Template
-TD-UPSE-B-AT
-CC BY-SA 4.0
-2019-01-17
-tall-dog.com</text>
-<text x="20" y="29" size="1.5" layer="22" ratio="10" rot="MR0" align="center">µPlaits SE
-Assembly Template
-TD-UPSE-B-AT
-CC BY-SA 4.0
-2019-01-17
-tall-dog.com</text>
+<text x="2" y="58.5" size="2" layer="22" ratio="12" rot="MR90" align="center">2021-01-01   tall-dog.com</text>
+<text x="20" y="10.75" size="2" layer="22" ratio="12" rot="MR180" align="center">TD-UPSE-C-AT</text>
 <hole x="7.5" y="96" drill="6.2"/>
 <hole x="7.5" y="81" drill="6.2"/>
@@
 <hole x="20" y="78" drill="3.2"/>
 <hole x="20" y="73" drill="3.2"/>
+<text x="38" y="58.5" size="2" layer="22" ratio="12" rot="MR270" align="center">µPlaits SE Assembly Template</text>
+<text x="20" y="26.5" size="3.5" layer="22" ratio="12" rot="MR0" align="center">2.0 mm</text>
+<text x="20" y="26.5" size="3.5" layer="21" ratio="12" align="center">2.0 mm</text>
+<wire x1="12" y1="29.5" x2="28" y2="29.5" width="0.254" layer="21"/>
+<wire x1="28" y1="29.5" x2="28" y2="23.5" width="0.254" layer="21"/>
+<wire x1="28" y1="23.5" x2="12" y2="23.5" width="0.254" layer="21"/>
+<wire x1="12" y1="23.5" x2="12" y2="29.5" width="0.254" layer="21"/>
+<wire x1="12" y1="29.5" x2="28" y2="29.5" width="0.254" layer="22"/>
+<wire x1="28" y1="29.5" x2="28" y2="23.5" width="0.254" layer="22"/>
+<wire x1="28" y1="23.5" x2="12" y2="23.5" width="0.254" layer="22"/>
+<wire x1="12" y1="23.5" x2="12" y2="29.5" width="0.254" layer="22"/>
+<text x="20" y="10.75" size="2" layer="21" ratio="12" rot="R180" align="center">TD-UPSE-C-AT</text>
+<text x="2" y="58.5" size="2" layer="21" ratio="12" rot="R270" align="center">µPlaits SE Assembly Template</text>
+<text x="38" y="58.5" size="2" layer="21" ratio="12" rot="R90" align="center">2021-01-01   tall-dog.com</text>
 </plain>
 <attributes>
@@
 <param name="mdSmdStop" value="0mil"/>
 <param name="msWidth" value="6mil"/>
-<param name="msDrill" value="0.35mm"/>
+<param name="msDrill" value="0.3mm"/>
 <param name="msMicroVia" value="9.99mm"/>
 <param name="msBlindViaRatio" value="0.5"/>
@@
 </autorouter>
 <elements>
+<element name="E$1" library="uPlaits_SE_Library" package="HOLE-M2.5" value="" x="20" y="67.5" smashed="yes"/>
+<element name="E$2" library="uPlaits_SE_Library" package="HOLE-M2.5" value="" x="20" y="4.5" smashed="yes"/>
 </elements>
 <signals>
-<signal name="S$1">
-<via x="20" y="67.5" extent="1-16" drill="2.75" diameter="5"/>
-</signal>
-<signal name="S$2">
-<via x="20" y="4.5" extent="1-16" drill="2.75" diameter="5"/>
+<signal name="GND">
+<polygon width="0.5" layer="1" isolate="0.5">
+<vertex x="0" y="110.5"/>
+<vertex x="40" y="110.5"/>
+<vertex x="40" y="0"/>
+<vertex x="0" y="0"/>
+</polygon>
+<polygon width="0.5" layer="16" isolate="0.5">
+<vertex x="0" y="110.5"/>
+<vertex x="40" y="110.5"/>
+<vertex x="40" y="0"/>
+<vertex x="0" y="0"/>
+</polygon>
 </signal>
 </signals>
@@
 <mfgpreviewcolor name="substratecolor" color="0xFF786E46"/>
 </mfgpreviewcolors>
+<errors>
+</errors>
 </board>
 </drawing>
-<compatibility>
-<note version="6.3" minversion="6.2.2" severity="warning">
-Since Version 6.2.2 text objects can contain more than one line,
-which will not be processed correctly with this version.
-</note>
-</compatibility>
 </eagle>

Commit message: updates and cleanup for Rev C production run
Other:
- board text added: "2024-07-06 tall-dog.com"
- board text added: "EITHER SIDE UP"
- board text removed: "2021-01-01 tall-dog.com"
Changed lines of the file:
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@@
 <setting verticaltext="up"/>
 </settings>
-<grid distance="0.5" unitdist="mm" unit="mm" style="lines" multiple="1" display="yes" altdistance="5" altunitdist="mil" altunit="mil"/>
+<grid distance="1" unitdist="mm" unit="mm" style="lines" multiple="1" display="yes" altdistance="5" altunitdist="mil" altunit="mil"/>
 <layers>
 <layer number="1" name="Top" color="4" fill="1" visible="yes" active="yes"/>
@@
 <wire x1="40" y1="3" x2="37" y2="0" width="0" layer="20" curve="-90"/>
 <wire x1="37" y1="110.5" x2="40" y2="107.5" width="0" layer="20" curve="-90"/>
-<text x="2" y="58.5" size="2" layer="22" ratio="12" rot="MR90" align="center">2021-01-01   tall-dog.com</text>
+<text x="2" y="58.5" size="2" layer="22" ratio="12" rot="MR90" align="center">2024-07-06   tall-dog.com</text>
 <text x="20" y="10.75" size="2" layer="22" ratio="12" rot="MR180" align="center">TD-UPSE-C-AT</text>
 <hole x="7.5" y="96" drill="6.2"/>
@@
 <hole x="20" y="73" drill="3.2"/>
 <text x="38" y="58.5" size="2" layer="22" ratio="12" rot="MR270" align="center">µPlaits SE Assembly Template</text>
-<text x="20" y="26.5" size="3.5" layer="22" ratio="12" rot="MR0" align="center">2.0 mm</text>
-<text x="20" y="26.5" size="3.5" layer="21" ratio="12" align="center">2.0 mm</text>
-<wire x1="12" y1="29.5" x2="28" y2="29.5" width="0.254" layer="21"/>
-<wire x1="28" y1="29.5" x2="28" y2="23.5" width="0.254" layer="21"/>
-<wire x1="28" y1="23.5" x2="12" y2="23.5" width="0.254" layer="21"/>
-<wire x1="12" y1="23.5" x2="12" y2="29.5" width="0.254" layer="21"/>
-<wire x1="12" y1="29.5" x2="28" y2="29.5" width="0.254" layer="22"/>
-<wire x1="28" y1="29.5" x2="28" y2="23.5" width="0.254" layer="22"/>
-<wire x1="28" y1="23.5" x2="12" y2="23.5" width="0.254" layer="22"/>
-<wire x1="12" y1="23.5" x2="12" y2="29.5" width="0.254" layer="22"/>
+<text x="20" y="30.5" size="3.5" layer="22" ratio="12" rot="MR0" align="center">2.0 mm</text>
+<text x="20" y="30.5" size="3.5" layer="21" ratio="12" align="center">2.0 mm</text>
+<wire x1="12" y1="33.5" x2="28" y2="33.5" width="0.254" layer="21"/>
+<wire x1="28" y1="33.5" x2="28" y2="27.5" width="0.254" layer="21"/>
+<wire x1="28" y1="27.5" x2="12" y2="27.5" width="0.254" layer="21"/>
+<wire x1="12" y1="27.5" x2="12" y2="33.5" width="0.254" layer="21"/>
+<wire x1="12" y1="33.5" x2="28" y2="33.5" width="0.254" layer="22"/>
+<wire x1="28" y1="33.5" x2="28" y2="27.5" width="0.254" layer="22"/>
+<wire x1="28" y1="27.5" x2="12" y2="27.5" width="0.254" layer="22"/>
+<wire x1="12" y1="27.5" x2="12" y2="33.5" width="0.254" layer="22"/>
 <text x="20" y="10.75" size="2" layer="21" ratio="12" rot="R180" align="center">TD-UPSE-C-AT</text>
 <text x="2" y="58.5" size="2" layer="21" ratio="12" rot="R270" align="center">µPlaits SE Assembly Template</text>
-<text x="38" y="58.5" size="2" layer="21" ratio="12" rot="R90" align="center">2021-01-01   tall-dog.com</text>
+<text x="38" y="58.5" size="2" layer="21" ratio="12" rot="R90" align="center">2024-07-06   tall-dog.com</text>
+<text x="20" y="24.5" size="2.5" layer="21" ratio="12" align="center">EITHER SIDE UP</text>
+<text x="20" y="24.5" size="2.5" layer="22" ratio="12" rot="MR0" align="center">EITHER SIDE UP</text>
 </plain>
 <attributes>
