File: uPlaits_SE_Control_Board.brd (EAGLE design)
At the start: 40 x 110.5 mm, 42 parts, among them J1 JACK-THONKICONN, J10 JACK-THONKICONN, J2 JACK-THONKICONN, J3 JACK-THONKICONN, J4 JACK-THONKICONN, J5 JACK-THONKICONN, J6 JACK-THONKICONN, J7 JACK-THONKICONN, J8 JACK-THONKICONN, J9 JACK-THONKICONN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

Commit message: updates and cleanup for Rev C production run
Parts:
- removed DS1, DS2, DS3, DS4, DS5, DS6, DS7, DS8: LED-SPACER, uPlaits_SE_Library:LED-SPACER
- added U$1: (no value), uPlaits_SE_Library:LED-SPACER
- P1, P2, P3, P4, P5, P6, P7: device uPlaits_SE_Library:POT-ALP-VERT-PS -> uPlaits_SE_Library:POT-SONG-9MM
Other:
- board text added: "CC BY-SA 4.0 2024-07-06 tall-dog.com"
- board text added: "TD-UPSE-C-CB"
- board text added: "uPlaits SE Control Board TD-UPSE-C-CB"
- board text added: "Émilie Gillet of Mutable Instruments"
- board text removed: "CC BY-SA 4.0 2019-02-18 tall-dog.com"
- board text removed: "Olivier Gillet of Mutable Instruments"
- board text removed: "TD- UPSE- B-CB"
- board text removed: "uPlaits SE Control Board TD-UPSE-B-CB"
