File: uPlaits_SE_Control_Board.sch (EAGLE design)
At the start: 42 parts, among them J1 JACK-THONKICONN, J10 JACK-THONKICONN, J2 JACK-THONKICONN, J3 JACK-THONKICONN, J4 JACK-THONKICONN, J5 JACK-THONKICONN, J6 JACK-THONKICONN, J7 JACK-THONKICONN, J8 JACK-THONKICONN, J9 JACK-THONKICONN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

Commit message: updates and cleanup for Rev C production run
Parts:
- removed DS1, DS2, DS3, DS4, DS5, DS6, DS7, DS8: LED-SPACER, uPlaits_SE_Library:LED-SPACER
Other:
- note added: "C"
- note removed: "B"
Changed lines of the file:
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@@
 <?xml version="1.0" encoding="utf-8"?>
 <!DOCTYPE eagle SYSTEM "eagle.dtd">
-<eagle version="9.3.0">
+<eagle version="9.6.2">
 <drawing>
 <settings>
@@
 <grid distance="0.1" unitdist="inch" unit="inch" style="lines" multiple="1" display="no" altdistance="0.01" altunitdist="inch" altunit="inch"/>
 <layers>
+<layer number="1" name="Top" color="4" fill="1" visible="no" active="no"/>
+<layer number="2" name="Route2" color="1" fill="3" visible="no" active="no"/>
+<layer number="3" name="Route3" color="4" fill="3" visible="no" active="no"/>
+<layer number="4" name="Route4" color="1" fill="4" visible="no" active="no"/>
+<layer number="5" name="Route5" color="4" fill="4" visible="no" active="no"/>
+<layer number="6" name="Route6" color="1" fill="8" visible="no" active="no"/>
+<layer number="7" name="Route7" color="4" fill="8" visible="no" active="no"/>
+<layer number="8" name="Route8" color="1" fill="2" visible="no" active="no"/>
+<layer number="9" name="Route9" color="4" fill="2" visible="no" active="no"/>
+<layer number="10" name="Route10" color="1" fill="7" visible="no" active="no"/>
+<layer number="11" name="Route11" color="4" fill="7" visible="no" active="no"/>
+<layer number="12" name="Route12" color="1" fill="5" visible="no" active="no"/>
+<layer number="13" name="Route13" color="4" fill="5" visible="no" active="no"/>
+<layer number="14" name="Route14" color="1" fill="6" visible="no" active="no"/>
+<layer number="15" name="Route15" color="4" fill="6" visible="no" active="no"/>
+<layer number="16" name="Bottom" color="1" fill="1" visible="no" active="no"/>
+<layer number="17" name="Pads" color="2" fill="1" visible="no" active="no"/>
+<layer number="18" name="Vias" color="2" fill="1" visible="no" active="no"/>
+<layer number="19" name="Unrouted" color="6" fill="1" visible="no" active="no"/>
+<layer number="20" name="Dimension" color="15" fill="1" visible="no" active="no"/>
+<layer number="21" name="tPlace" color="7" fill="1" visible="no" active="no"/>
+<layer number="22" name="bPlace" color="7" fill="1" visible="no" active="no"/>
+<layer number="23" name="tOrigins" color="15" fill="1" visible="no" active="no"/>
+<layer number="24" name="bOrigins" color="15" fill="1" visible="no" active="no"/>
+<layer number="25" name="tNames" color="7" fill="1" visible="no" active="no"/>
+<layer number="26" name="bNames" color="7" fill="1" visible="no" active="no"/>
+<layer number="27" name="tValues" color="7" fill="1" visible="no" active="no"/>
+<layer number="28" name="bValues" color="7" fill="1" visible="no" active="no"/>
+<layer number="29" name="tStop" color="7" fill="3" visible="no" active="no"/>
+<layer number="30" name="bStop" color="7" fill="6" visible="no" active="no"/>
+<layer number="31" name="tCream" color="7" fill="4" visible="no" active="no"/>
+<layer number="32" name="bCream" color="7" fill="5" visible="no" active="no"/>
+<layer number="33" name="tFinish" color="6" fill="3" visible="no" active="no"/>
+<layer number="34" name="bFinish" color="6" fill="6" visible="no" active="no"/>
+<layer number="35" name="tGlue" color="7" fill="4" visible="no" active="no"/>
+<layer number="36" name="bGlue" color="7" fill="5" visible="no" active="no"/>
+<layer number="37" name="tTest" color="7" fill="1" visible="no" active="no"/>
+<layer number="38" name="bTest" color="7" fill="1" visible="no" active="no"/>
+<layer number="39" name="tKeepout" color="4" fill="11" visible="no" active="no"/>
+<layer number="40" name="bKeepout" color="1" fill="11" visible="no" active="no"/>
+<layer number="41" name="tRestrict" color="4" fill="10" visible="no" active="no"/>
+<layer number="42" name="bRestrict" color="1" fill="10" visible="no" active="no"/>
+<layer number="43" name="vRestrict" color="2" fill="10" visible="no" active="no"/>
+<layer number="44" name="Drills" color="7" fill="1" visible="no" active="no"/>
+<layer number="45" name="Holes" color="7" fill="1" visible="no" active="no"/>
+<layer number="46" name="Milling" color="3" fill="1" visible="no" active="no"/>
+<layer number="47" name="Measures" color="7" fill="1" visible="no" active="no"/>
+<layer number="48" name="Document" color="7" fill="1" visible="no" active="no"/>
+<layer number="49" name="Reference" color="7" fill="1" visible="no" active="no"/>
+<layer number="51" name="tDocu" color="7" fill="1" visible="no" active="no"/>
+<layer number="52" name="bDocu" color="7" fill="1" visible="no" active="no"/>
 <layer number="88" name="SimResults" color="9" fill="1" visible="yes" active="yes"/>
 <layer number="89" name="SimProbes" color="9" fill="1" visible="yes" active="yes"/>
@@
 <part name="D7" library="uPlaits_SE_Library" deviceset="LED-DUAL" device="-PTH"/>
 <part name="D8" library="uPlaits_SE_Library" deviceset="LED-DUAL" device="-PTH"/>
-<part name="DS1" library="uPlaits_SE_Library" deviceset="LED-SPACER" device=""/>
-<part name="DS2" library="uPlaits_SE_Library" deviceset="LED-SPACER" device=""/>
-<part name="DS3" library="uPlaits_SE_Library" deviceset="LED-SPACER" device=""/>
-<part name="DS4" library="uPlaits_SE_Library" deviceset="LED-SPACER" device=""/>
-<part name="DS5" library="uPlaits_SE_Library" deviceset="LED-SPACER" device=""/>
-<part name="DS6" library="uPlaits_SE_Library" deviceset="LED-SPACER" device=""/>
-<part name="DS7" library="uPlaits_SE_Library" deviceset="LED-SPACER" device=""/>
-<part name="DS8" library="uPlaits_SE_Library" deviceset="LED-SPACER" device=""/>
 <part name="P1" library="uPlaits_SE_Library" deviceset="POT" device="-ALPS-VERT-PS" value="B10k"/>
 <part name="P2" library="uPlaits_SE_Library" deviceset="POT" device="-ALPS-VERT-PS" value="B10k"/>
@@
 Olivier Gillet of Mutable Instruments</text>
 <text x="148.59" y="6.35" size="2.54" layer="94">Website: tall-dog.com</text>
-<text x="236.22" y="6.35" size="3.81" layer="94">B</text>
+<text x="236.22" y="6.35" size="3.81" layer="94">C</text>
 <text x="179.07" y="11.43" size="2.54" layer="94">N/A</text>
 <text x="247.65" y="19.05" size="3.81" layer="94" align="center-right">Control Board</text>
@@
 <attribute name="NAME" x="196.85" y="116.84" size="1.524" layer="95" rot="MR180" align="center-left"/>
 </instance>
-<instance part="DS1" gate="G$1" x="213.36" y="66.04" smashed="yes" rot="R90">
-<attribute name="NAME" x="218.44" y="66.04" size="1.524" layer="95" rot="R270" align="center"/>
-</instance>
-<instance part="DS2" gate="G$1" x="213.36" y="78.74" smashed="yes" rot="R90">
-<attribute name="NAME" x="218.44" y="78.74" size="1.524" layer="95" rot="R270" align="center"/>
-</instance>
-<instance part="DS3" gate="G$1" x="213.36" y="91.44" smashed="yes" rot="R90">
-<attribute name="NAME" x="218.44" y="91.44" size="1.524" layer="95" rot="R270" align="center"/>
-</instance>
-<instance part="DS4" gate="G$1" x="213.36" y="104.14" smashed="yes" rot="R90">
-<attribute name="NAME" x="218.44" y="104.14" size="1.524" layer="95" rot="R270" align="center"/>
-</instance>
-<instance part="DS5" gate="G$1" x="213.36" y="154.94" smashed="yes" rot="R90">
-<attribute name="NAME" x="218.44" y="154.94" size="1.524" layer="95" rot="R270" align="center"/>
-</instance>
-<instance part="DS6" gate="G$1" x="213.36" y="142.24" smashed="yes" rot="R90">
-<attribute name="NAME" x="218.44" y="142.24" size="1.524" layer="95" rot="R270" align="center"/>
-</instance>
-<instance part="DS7" gate="G$1" x="213.36" y="129.54" smashed="yes" rot="R90">
-<attribute name="NAME" x="218.44" y="129.54" size="1.524" layer="95" rot="R270" align="center"/>
-</instance>
-<instance part="DS8" gate="G$1" x="213.36" y="116.84" smashed="yes" rot="R90">
-<attribute name="NAME" x="218.44" y="116.84" size="1.524" layer="95" rot="R270" align="center"/>
-</instance>
 <instance part="P1" gate="G$1" x="147.32" y="149.86" smashed="yes">
