File: uPlaits_SE_Front_Panel.brd (EAGLE design)
At the start: 40.3 x 128.5 mm, 2 parts

Commit message: updates and cleanup for Rev C production run
Other:
- board text added: "Panel derived from work by Émilie Gillet of Mutable Instruments"
- board text added: "TD-UPSE-C"
- board text added: "µPlaits SE Front Panel TD-UPSE-C-FP CC BY-SA 4.0 2024-07-06 tall-dog.com"
- board text removed: "Panel derived from work by Olivier Gillet of Mutable Instruments"
- board text removed: "TD-UPSE-B"
- board text removed: "µPlaits SE Front Panel TD-UPSE-B-FP CC BY-SA 4.0 2019-01-17 tall-dog.com"
Changed lines of the file:
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@@
 <?xml version="1.0" encoding="utf-8"?>
 <!DOCTYPE eagle SYSTEM "eagle.dtd">
-<eagle version="9.3.0">
+<eagle version="9.6.2">
 <drawing>
 <settings>
@@
 <text x="20.15" y="39" size="1.5" layer="30" ratio="10" rot="MR0" align="center">µPlaits SE
 Front Panel
-TD-UPSE-B-FP
+TD-UPSE-C-FP
 CC BY-SA 4.0
-2019-01-17
+2024-07-06
 tall-dog.com</text>
 <text x="20.15" y="1.5" size="1.5" layer="30" ratio="10" rot="MR0" align="bottom-center">Panel
 derived
 from work by
-Olivier Gillet
+Émilie Gillet
 of Mutable
 Instruments</text>
-<text x="20.15" y="125.5" size="1.5" layer="29" ratio="10" align="center">TD-UPSE-B</text>
+<text x="20.15" y="125.5" size="1.5" layer="29" ratio="10" align="center">TD-UPSE-C</text>
 <wire x1="13.4" y1="127" x2="26.9" y2="127" width="0.15" layer="29"/>
 <wire x1="26.9" y1="127" x2="26.9" y2="124" width="0.15" layer="29"/>
