File: uPlaits_SE_Main_Board.brd (EAGLE design)
At the start: 40 x 110.5 mm, 141 parts, among them U1 MCP6004-TSSOP-14, U2 MCP6004-TSSOP-14, U3 TLC59281-SSOP-24, U4 STM32F373-LQFP-48, U5 TL072-SO-8, U6 PCM5100A-TSSOP-20, U7 LM4040-SOT-23, U8 REG-SOT-23-5, U9 REG-R-78E, X1 8MHz

Commit message: updates and cleanup for Rev C production run
Parts:
- removed U$2: (no value), uPlaits_SE_Library:TALL-DOG-LOGO-INVERT
- removed U$3, U$5: (no value), uRings_SE_Library:MARKING-OSH-LOGO-5MM
- removed U$4: (no value), uRings_SE_Library:MARKING-CC-LOGO
- added U$10: (no value), uPlaits_SE_Library:LOGO-OSH
- added U$11: (no value), uPlaits_SE_Library:LOGO-OSHW
- added U$12: (no value), uPlaits_SE_Library:LOGO-PN
- added U$13: (no value), uPlaits_SE_Library:LOGO-QC
- added U$14: (no value), uPlaits_SE_Library:LOGO-REV
- added U$15: (no value), uPlaits_SE_Library:LOGO-SN
- added U$9: (no value), uPlaits_SE_Library:LOGO-CC
- D1, D2, D3, D4, D5, D6, D7, D8: value (none) -> TVS-0603
- U$1: device uRings_SE_Library:MARKING-CC-LOGO -> uPlaits_SE_Library:LOGO-TD
- moved U$1 18.2 mm to (26.5, 98.5), turned to 0 degrees
Other:
- board text added: "Board derived from work by Émilie Gillet of Mutable Instruments"
- board text added: "TD-UPSE-C-MB 2024-07-06"
- board text removed: "BY-SA 4.0"
- board text removed: "Board derived from work by Olivier Gillet of Mutable Instruments"
- board text removed: "SN"
- board text removed: "TD-UPSE-B 2019-01-17 tall-dog.com"
- board text removed: "TD-UPSE-B-MB"
- board text removed: "open source hardware"
- board text removed: "uPlaits SE Main Board TD-UPSE-B-MB CC BY-SA 4.0 2019-01-17 tall-dog.com"
- board text removed: "µPlaits SE"
