File: uPlaits_SE_Main_Board.sch (EAGLE design)
At the start: 133 parts, among them U1 MCP6004-TSSOP-14, U2 MCP6004-TSSOP-14, U3 TLC59281-SSOP-24, U4 STM32F373-LQFP-48, U5 TL072-SO-8, U6 PCM5100A-TSSOP-20, U7 LM4040-SOT-23, U8 REG-SOT-23-5, U9 REG-R-78E, X1 8MHz

Commit message: updates and cleanup for Rev C production run
Other:
- note added: "C"
- note removed: "B"
